File: RB-347.kicad_sch (KiCad schematic)
At the start: 31 parts, among them J1 Conn_USB_C_Socket, J2 PINHD_1x10_Male, J3 PINHD_1x10_Male, J4 PINHD_1x10_Male, SW1 I2C, SW2 SPDT_Slide_SMD_6.7x2.6mm, U1 USBLC6-2SC6, U2 CH347F, U3 TLV74333PDBVR, U4 TLV74318PDBVR, Y1 8Mhz

Commit message: add I²C indicator LED
Parts:
- added LED2: POWER, PCM_SparkFun-LED:LED_0402_1005Metric_Red, symbol PCM_LED_AKL:LED_0402_Red
- added R8: 1k, Resistor_SMD:R_0402_1005Metric, symbol PCM_SparkFun-Resistor:5.1k_0603
- R1: now not fitted
- renumbered R9 to R10, R8 to R9
Connections:
- net GND: now also LED2.1 (K)
- net at R10.1, R9.1, SW1.1: now also R8.2
- new net: LED2.2 (A), R8.1
